File: STM32F446RE minsys.kicad_sch (KiCad schematic)
At the start: 37 parts, among them J1 USB_B_Mini, J2 ST-LINKV2, J3 Conn_02x13_Odd_Even, J4 Conn_02x12_Odd_Even, J5 Conn_02x12_Odd_Even, J6 Conn_02x12_Odd_Even, SW1 SW_SPST, U1 STM32F446RETx, U2 TPS79533DCQ, Y1 8.192MHz

Commit message: Sync Tractor VCU project and manufacturing exports
Update KiCad project files, drill maps, BOM, STEP, and ODB++ exports from the source project. Replace the Gerber directory with the original Gerber.zip archive and remove obsolete drill outputs.
Parts:
- renumbered C9 to C10, C10 to C11, C11 to C12, C12 to C13, C13 to C14, C14 to C15, C15 to C6, C6 to C7, C7 to C8, C8 to C9, R2 to R1, R4 to R2, R5 to R3, R7 to R4, R1 to R5, R6 to R62, U2 to U1, U1 to U2
