File: Tractor VCU.kicad_pcb (KiCad board)
At the start: 4 copper layers, 180 x 180 mm, 208 parts, among them J1 USB_B_Mini, J10 PUMP MOTOR, J11 BRAKE1, J12 BRAKE2, J13 CAN_MCP2551, J14 CAN_MCP2551, J15 CAN1 TEST, J16 CAN2 TEST, J17 SD CARD MODULE, J18 USART, J19 ADC1_IN12, J2 ST-LINKV2, J20 ADC1_IN13, J21 INPUT, J3 Conn_02x13_Odd_Even, J4 Conn_02x12_Odd_Even, J5 Conn_02x12_Odd_Even, J6 Conn_02x12_Odd_Even, J7 RELAY1_EXTERNAL, J8 RELAY2_EXTERNAL, J9 MAIN MOTOR, K1 RELAY_MM, K10 RELAY_PM, K11 RELAY_EX, K12 RELAY_EX, K2 RELAY_MM, K3 RELAY_MM, K4 RELAY_MM, K5 RELAY_MM, K6 RELAY_PM, K7 RELAY_PM, K8 RELAY_PM, K9 RELAY_PM, Q1 BC846, Q10 BC846, Q11 BC846, Q12 BC846, Q13 GT6K2P10KH, Q2 BC846, Q3 BC846, Q4 BC846, Q5 BC846, Q6 BC846, Q7 BC846, Q8 BC846, Q9 BC846, SW1 SW_SPST, SW2 SW_SPDT, U1 TPS79533DCQ, U2 STM32F446RETx, U3 LM358, U4 TPS79533DCQ, Y1 8.192MHz

Commit message: Sync Tractor VCU project and manufacturing exports
Update KiCad project files, drill maps, BOM, STEP, and ODB++ exports from the source project. Replace the Gerber directory with the original Gerber.zip archive and remove obsolete drill outputs.
Parts:
- J15, J16, J7, J8: footprint Connector_Wuerth:Wuerth 691137710002_1x02 -> Connector_Wuerth:Wuerth_TBL_691137710002_1x02_P5mm
