File: VCU Connectors.kicad_sch (KiCad schematic)
At the start: 49 parts, among them J10 PUMP MOTOR, J11 BRAKE1, J12 BRAKE2, J13 CAN_MCP2551, J14 CAN_MCP2551, J15 CAN1 TEST, J16 CAN2 TEST, J17 SD CARD MODULE, J18 USART, J19 ADC1_IN12, J20 ADC1_IN13, J9 MAIN MOTOR, U3 LM358

Commit message: Sync Tractor VCU project and manufacturing exports
Update KiCad project files, drill maps, BOM, STEP, and ODB++ exports from the source project. Replace the Gerber directory with the original Gerber.zip archive and remove obsolete drill outputs.
Parts:
- J15, J16: footprint Connector_Wuerth:Wuerth 691137710002_1x02 -> Connector_Wuerth:Wuerth_TBL_691137710002_1x02_P5mm
