File: VCU Relays.kicad_sch (KiCad schematic)
At the start: 86 parts, among them J7 RELAY1_EXTERNAL, J8 RELAY2_EXTERNAL, K1 RELAY_MM, K10 RELAY_PM, K11 RELAY_EX, K12 RELAY_EX, K2 RELAY_MM, K3 RELAY_MM, K4 RELAY_MM, K5 RELAY_MM, K6 RELAY_PM, K7 RELAY_PM, K8 RELAY_PM, K9 RELAY_PM, Q1 BC846, Q10 BC846, Q11 BC846, Q12 BC846, Q2 BC846, Q3 BC846, Q4 BC846, Q5 BC846, Q6 BC846, Q7 BC846, Q8 BC846, Q9 BC846

Commit message: Sync Tractor VCU project and manufacturing exports
Update KiCad project files, drill maps, BOM, STEP, and ODB++ exports from the source project. Replace the Gerber directory with the original Gerber.zip archive and remove obsolete drill outputs.
Parts:
- J7, J8: footprint Connector_Wuerth:Wuerth 691137710002_1x02 -> Connector_Wuerth:Wuerth_TBL_691137710002_1x02_P5mm
