File: power supply.kicad_sch (KiCad schematic)
At the start: 35 parts, among them SW2 SW_SPDT

Commit message: Sync Tractor VCU project and manufacturing exports
Update KiCad project files, drill maps, BOM, STEP, and ODB++ exports from the source project. Replace the Gerber directory with the original Gerber.zip archive and remove obsolete drill outputs.
Parts:
- gave numbers to parts that had none: 22
